Commit message: feat: 新增chassis_control移动底盘包(PS100驱动/ChassisMove服务/站间移动)与任务区物料区动作配置，Teensy驱动重构支持calibrate与serial_port参数

File: ros2/src/ar_description/urdf/ar_macro.xacro (robot description, xacro)
@@ -85,5 +85,5 @@
       <child link="link_2"/>
       <axis xyz="0 0 -1"/>
-      <limit lower="${-42.0 / 180.0 * pi}" upper="${90.0 / 180.0 * pi}" effort="0.5" velocity="0"/>
+      <limit lower="${-36.0 / 180.0 * pi}" upper="${96.0 / 180.0 * pi}" effort="0.5" velocity="0"/>
     </joint>
     <link name="link_3">
